File: pcb/purple-eye.sch (EAGLE design)
At the start: 10 parts

Commit message: feat: add charging circuit
Parts:
- added C1: 4.7uF, SparkFun-Capacitors:4.7UF-6.3V-10%(0603)0603
- added D1: RED, SparkFun-LED:LED-RED0603
- added J7: USB-MICROB, SparkFun-Connectors:USB-MICROB
- added R3: 2.0k, SparkFun-Resistors:2.0KOHM1/10W5%(0603)
- added R4: 4.7K, SparkFun-Resistors:4.7KOHM-1/10W-1%(0603)
- added U1: MCP73831, SparkFun-PowerIC:MCP73831
- R1, R2: value 10k -> 10K; device SparkFun-Resistors:10KOHM-1/4W5%(PTH)HORIZ-KIT -> SparkFun-Resistors:10KOHM-1/10W-1%(0603)0603
Connections:
- new net N$3: D1.A, R4.1
- new net N$4: D1.C, U1.STAT
- new net VBAT: J1.2, S1.O, U1.VBAT
- new net VBUS: C1.2, J7.VBUS, R4.2, U1.VIN
- net GND: now also C1.1, J7.GND, R3.2, U1.VSS
- net N$2: now also R3.1, U1.PROG; no longer J1.2, S1.O
Other:
- note added: "Charging"
- moved on the sheet: J1, S1
Changed lines of the file:
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@@
 <parts>
 <part name="JP6" library="SparkFun-Connectors" deviceset="M02" device="LOCK"/>
-<part name="R1" library="SparkFun-Resistors" deviceset="10KOHM-1/4W5%(PTH)" device="HORIZ-KIT" value="10k"/>
-<part name="R2" library="SparkFun-Resistors" deviceset="10KOHM-1/4W5%(PTH)" device="HORIZ-KIT" value="10k"/>
+<part name="R1" library="SparkFun-Resistors" deviceset="10KOHM-1/10W-1%(0603)" device="0603" value="10K"/>
+<part name="R2" library="SparkFun-Resistors" deviceset="10KOHM-1/10W-1%(0603)" device="0603" value="10K"/>
 <part name="S1" library="SparkFun-Electromechanical" deviceset="SWITCH-SPDT" device="PTH_LOCK"/>
 <part name="GND1" library="supply1" deviceset="GND" device=""/>
@@
 <part name="J5" library="SparkFun-Connectors" deviceset="M03" device="LOCK"/>
 <part name="J6" library="SparkFun-Connectors" deviceset="M05" device="LOCK"/>
+<part name="U1" library="SparkFun-PowerIC" deviceset="MCP73831" device=""/>
+<part name="GND8" library="supply1" deviceset="GND" device=""/>
+<part name="R3" library="SparkFun-Resistors" deviceset="2.0KOHM1/10W5%(0603)" device="" value="2.0k"/>
+<part name="GND9" library="supply1" deviceset="GND" device=""/>
+<part name="J7" library="SparkFun-Connectors" deviceset="USB" device="-MICROB"/>
+<part name="GND10" library="supply1" deviceset="GND" device=""/>
+<part name="C1" library="SparkFun-Capacitors" deviceset="4.7UF-6.3V-10%(0603)" device="0603" value="4.7uF"/>
+<part name="GND11" library="supply1" deviceset="GND" device=""/>
+<part name="D1" library="SparkFun-LED" deviceset="LED-RED" device="0603" value="RED"/>
+<part name="R4" library="SparkFun-Resistors" deviceset="4.7KOHM-1/10W-1%(0603)" device="" value="4.7K"/>
 </parts>
 <sheets>
 <sheet>
 <plain>
+<text x="22.86" y="119.38" size="1.778" layer="91">Charging</text>
 </plain>
 <instances>
@@
 <instance part="R1" gate="G$1" x="-20.32" y="78.74"/>
 <instance part="R2" gate="G$1" x="-38.1" y="83.82"/>
-<instance part="S1" gate="1" x="50.8" y="86.36" rot="R90"/>
+<instance part="S1" gate="1" x="53.34" y="76.2" rot="R90"/>
 <instance part="GND1" gate="1" x="-30.48" y="58.42" rot="R270"/>
 <instance part="GND2" gate="1" x="17.78" y="58.42" rot="R270"/>
@@
 <instance part="GND4" gate="1" x="17.78" y="38.1" rot="R270"/>
 <instance part="GND5" gate="1" x="-30.48" y="22.86" rot="R270"/>
-<instance part="GND6" gate="1" x="38.1" y="88.9" rot="R90"/>
+<instance part="GND6" gate="1" x="40.64" y="78.74" rot="R90"/>
 <instance part="GND7" gate="1" x="-48.26" y="81.28"/>
-<instance part="J1" gate="G$1" x="22.86" y="88.9"/>
+<instance part="J1" gate="G$1" x="25.4" y="78.74"/>
 <instance part="J2" gate="J$1" x="5.08" y="55.88" rot="R180"/>
 <instance part="J3" gate="J$1" x="5.08" y="38.1" rot="R180"/>
@@
 <instance part="J5" gate="J$1" x="43.18" y="55.88" rot="R180"/>
 <instance part="J6" gate="G$1" x="5.08" y="88.9" rot="R180"/>
+<instance part="U1" gate="G$1" x="30.48" y="109.22"/>
+<instance part="GND8" gate="1" x="48.26" y="104.14"/>
+<instance part="R3" gate="G$1" x="58.42" y="109.22"/>
+<instance part="GND9" gate="1" x="68.58" y="109.22" rot="R90"/>
+<instance part="J7" gate="G$1" x="-27.94" y="114.3" rot="R180"/>
+<instance part="GND10" gate="1" x="-17.78" y="119.38" rot="R180"/>
+<instance part="C1" gate="G$1" x="0" y="111.76" rot="R90"/>
+<instance part="GND11" gate="1" x="-5.08" y="106.68"/>
+<instance part="D1" gate="G$1" x="12.7" y="101.6" rot="R90"/>
+<instance part="R4" gate="G$1" x="5.08" y="106.68" rot="R90"/>
 </instances>
 <busses>
@@
 <segment>
 <pinref part="GND6" gate="1" pin="GND"/>
-<wire x1="35.56" y1="88.9" x2="30.48" y2="88.9" width="0.1524" layer="91"/>
+<wire x1="38.1" y1="78.74" x2="33.02" y2="78.74" width="0.1524" layer="91"/>
 <pinref part="J1" gate="G$1" pin="1"/>
 </segment>
@@
 <pinref part="J5" gate="J$1" pin="1"/>
 </segment>
+<segment>
+<pinref part="U1" gate="G$1" pin="VSS"/>
+<pinref part="GND8" gate="1" pin="GND"/>
+<wire x1="40.64" y1="106.68" x2="48.26" y2="106.68" width="0.1524" layer="91"/>
+</segment>
+<segment>
+<pinref part="R3" gate="G$1" pin="2"/>
+<pinref part="GND9" gate="1" pin="GND"/>
+<wire x1="63.5" y1="109.22" x2="66.04" y2="109.22" width="0.1524" layer="91"/>
+</segment>
+<segment>
+<pinref part="J7" gate="G$1" pin="GND"/>
+<pinref part="GND10" gate="1" pin="GND"/>
+<wire x1="-25.4" y1="114.3" x2="-17.78" y2="114.3" width="0.1524" layer="91"/>
+<wire x1="-17.78" y1="114.3" x2="-17.78" y2="116.84" width="0.1524" layer="91"/>
+</segment>
+<segment>
+<pinref part="GND11" gate="1" pin="GND"/>
+<pinref part="C1" gate="G$1" pin="1"/>
+<wire x1="-5.08" y1="109.22" x2="-5.08" y2="111.76" width="0.1524" layer="91"/>
+</segment>
 </net>
 <net name="VCC" class="0">
@@
 <segment>
 <pinref part="S1" gate="1" pin="P"/>
-<wire x1="50.8" y1="83.82" x2="73.66" y2="83.82" width="0.1524" layer="91"/>
-<label x="71.12" y="83.82" size="1.778" layer="95"/>
+<wire x1="53.34" y1="73.66" x2="76.2" y2="73.66" width="0.1524" layer="91"/>
+<label x="73.66" y="73.66" size="1.778" layer="95"/>
 </segment>
 <segment>
@@
 <segment>
 <pinref part="R1" gate="G$1" pin="1"/>
-<wire x1="-25.4" y1="78.74" x2="-25.4" y2="73.66" width="0.1524" layer="91"/>
-<label x="-25.4" y="73.66" size="1.778" layer="95"/>
+<wire x1="-25.4" y1="78.74" x2="-33.02" y2="78.74" width="0.1524" layer="91"/>
+<label x="-33.02" y="78.74" size="1.778" layer="95"/>
 </segment>
 </net>
@@
 </segment>
 </net>
-<net name="N$2" class="0">
+<net name="VBAT" class="0">
+<segment>
+<pinref part="U1" gate="G$1" pin="VBAT"/>
+<wire x1="40.64" y1="111.76" x2="50.8" y2="111.76" width="0.1524" layer="91"/>
+<label x="45.72" y="111.76" size="1.778" layer="95"/>
+</segment>
 <segment>
 <pinref part="J1" gate="G$1" pin="2"/>
 <pinref part="S1" gate="1" pin="O"/>
-<wire x1="30.48" y1="91.44" x2="48.26" y2="91.44" width="0.1524" layer="91"/>
-</segment>
-</net>
+<wire x1="33.02" y1="81.28" x2="50.8" y2="81.28" width="0.1524" layer="91"/>
+<label x="35.56" y="81.28" size="1.778" layer="95"/>
+</segment>
+</net>
+<net name="N$2" class="0">
+<segment>
+<pinref part="U1" gate="G$1" pin="PROG"/>
+<pinref part="R3" gate="G$1" pin="1"/>
+<wire x1="40.64" y1="109.22" x2="53.34" y2="109.22" width="0.1524" layer="91"/>
+</segment>
+</net>
+<net name="VBUS" class="0">
+<segment>
+<pinref part="J7" gate="G$1" pin="VBUS"/>
+<wire x1="-25.4" y1="111.76" x2="-15.24" y2="111.76" width="0.1524" layer="91"/>
+<label x="-20.32" y="111.76" size="1.778" layer="95"/>
+</segment>
+<segment>
+<pinref part="U1" gate="G$1" pin="VIN"/>
+<wire x1="20.32" y1="111.76" x2="5.08" y2="111.76" width="0.1524" layer="91"/>
+<pinref part="C1" gate="G$1" pin="2"/>
+<label x="12.7" y="111.76" size="1.778" layer="95"/>
+<pinref part="R4" gate="G$1" pin="2"/>
+<wire x1="5.08" y1="111.76" x2="2.54" y2="111.76" width="0.1524" layer="91"/>
+<junction x="5.08" y="111.76"/>
+</segment>
+</net>
+<net name="N$3" class="0">
+<segment>
+<pinref part="D1" gate="G$1" pin="A"/>
+<pinref part="R4" gate="G$1" pin="1"/>
+<wire x1="10.16" y1="101.6" x2="5.08" y2="101.6" width="0.1524" layer="91"/>
+</segment>
+</net>
+<net name="N$4" class="0">
+<segment>
+<pinref part="U1" gate="G$1" pin="STAT"/>
+<wire x1="20.32" y1="106.68" x2="20.32" y2="101.6" width="0.1524" layer="91"/>
+<pinref part="D1" gate="G$1" pin="C"/>
+<wire x1="20.32" y1="101.6" x2="17.78" y2="101.6" width="0.1524" layer="91"/>
+</segment>
+</net>
